File: Headpho.kicad_pcb (KiCad board)
At the start: 2 copper layers, 45.6 x 128.5 mm, 45 parts, among them IC1 NJM4556AD, IC2 NJM4556AD, J1 IN L, J2 IN R, J3 Eurorack_Power_10pin_Unshroud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, J4 LINE OUT L, J5 OUT LR, J6 LINE OUT R, U1 LME49720, U2 LME49720

Commit message: v1.0 almost ready for production
Parts:
- removed REF** (x5): GND, PCM_4ms_Faceplate:Faceplate_Hole_Jack_3.5mm
- removed REF**: Faceplate_Hole_Pot_9mm, PCM_4ms_Faceplate:Faceplate_Hole_Pot_9mm
- C1, C2: value 22u -> 22uF
- C10, C9: value 104▶ -> 100n
- C11, C12: value 220 -> 22p
- C13, C14, C3, C4, C5, C6, C7, C8: value 104 -> 100n
- R1, R2: value 100k▶ -> 100k
- moved C2 1.49 mm to (68.1, 94.7), turned to 90 degrees
Connections:
- J2 pad 1: unconnected-(J2-SIG-Pad1) -> Net-(J2-SIG)
- POT1 pad 7: (no net) -> unconnected-(POT1C-SHELL-2-Pad7)
- POT1 pad 8: (no net) -> unconnected-(POT1C-SHELL-1-Pad8)
- R1 pad 1: Net-(U1A--) -> Net-(J1-SIG)
- R2 pad 1: Net-(U1B--) -> Net-(J2-SIG)
- U1 pad 2: Net-(U1A--) -> Net-(J1-SIG)
- U1 pad 6: Net-(U1B--) -> Net-(J2-SIG)
Routing:
- net Net-(J2-SIG): track 0.00 -> 23.7 mm
- net Net-(J1-SIG): track 13.7 -> 36.9 mm
- net Net-(J6-SIG): track 92.1 -> 106.8 mm, vias 2 -> 0
- net Net-(IC1-A_+INPUT): track 52.6 -> 63.2 mm, vias 0 -> 2
- net Net-(U1A--): track 8.92 -> 0.00 mm
- net Net-(U1B--): track 6.23 -> 0.00 mm
- net +12V: track 78.5 -> 83.7 mm
- net Net-(J5-SIG): track 28.4 -> 24.0 mm
- net Net-(R1-Pad2): track 22.5 -> 18.3 mm
- net Net-(C12-Pad2): track 14.9 -> 18.6 mm
- net Net-(IC1-A_-INPUT): track 21.0 -> 17.2 mm
- net Net-(J4-SIG): track 72.1 -> 68.6 mm, vias 3 -> 2
- net -12V: track 88.2 -> 90.1 mm
- net Net-(U2A--): track 11.5 -> 13.3 mm
- net Net-(IC1-B_-INPUT): track 8.54 -> 7.25 mm, vias 1 -> 0
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Other:
- board size 45.6 x 128.5 mm -> 20 x 106.7 mm
- board text added: "INSPIRED BY: RAMPHANDS EXITS & FORESTCAVER AJH"
- board text added: "JLCJLCJLCJLC"
- board text added: "PCB BY 42 BERLIN SYNTHLAB"
- board text added: "STEREO HEADPHONE AMP"
- board text added: "V1.0"
- board text added: "`HEADPHO`"
- board text added: "https://www.github.com/ fablabnk/SynthLabProjects"
- board text removed: "HEAD PHO"
- board text removed: "IN L"
- board text removed: "IN R"
- board text removed: "LINE"
- board text removed: "OUT L"
- board text removed: "OUT R"
- board text removed: "PHONES OUT"
- board text removed: "VOLUME"
- board text removed: "▶"
