File: Headpho.kicad_sch (KiCad schematic)
At the start: 39 parts, among them IC1 NJM4556AD, IC2 NJM4556AD, J1 IN L, J2 IN R, J3 Eurorack_Power_10pin_Unshroud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, J4 LINE OUT L, J5 OUT LR, J6 LINE OUT R, U1 LME49720, U2 LME49720

Commit message: v1.0 almost ready for production
Parts:
- removed IC1, IC2: NJM4556AD, Package_DIP:DIP-8_W7.62mm_Socket, symbol SamacSys_Parts:NJM4556AV-TE1
- added IC1, IC2: NJM4556AD, Package_DIP:DIP-8_W7.62mm_Socket, symbol Library:NJM4556AV-TE1
- added unit 3 of POT1
- C1, C2: value 22u -> 22uF
- C10, C9: value 104 -> 100n; Silkscreen Value (none) -> 104▶
- C11, C12: value 220 -> 22p; Silkscreen Value (none) -> ▼220
- C13, C4, C6, C7, C8: value 104 -> 100n; Silkscreen Value (none) -> 104▼
- C14: value 104 -> 100n; Silkscreen Value (none) -> ▲104
- C3, C5: value 104 -> 100n; Silkscreen Value (none) -> 104▲
Connections:
- net +12V: now also IC1.8 (V+), IC2.8 (V+)
- net -12V: now also IC1.4 (V-), IC2.4 (V-)
- net at J1.1 (SIG), J2.3 (SW): now also R1.1, U1.2 (-)
- net at C14.2, R10.2: now also IC2.3 (A_+INPUT), IC2.5 (B_+INPUT)
- net at J2.1 (SIG): now also R2.1, U1.6 (-)
- net at R11.1: now also IC1.1 (A_OUTPUT), IC1.2 (A_-INPUT)
- net at C13.2, R9.2: now also IC1.3 (A_+INPUT), IC1.5 (B_+INPUT)
- net at R12.1: now also IC1.6 (B_-INPUT), IC1.7 (B_OUTPUT)
- net at R13.1: now also IC2.1 (A_OUTPUT), IC2.2 (A_-INPUT)
- net at R14.1: now also IC2.6 (B_-INPUT), IC2.7 (B_OUTPUT)
- no-connect marks 3 -> 5

Commit message: v1.0 ready for production - fixed some minor silkscreening issues such as adding arrows
Parts:
- C1: Silkscreen Value (none) -> 22uF▶
- C2: Silkscreen Value (none) -> ◀22uF
- R1, R2: Silkscreen Value (none) -> 100k▶
Changed lines of the file:
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@@
+			)
+		)
+		(property "Silkscreen Value" "100k▶"
+			(at 53.34 57.15 90)
+			(effects
+				(font
+					(size 1.27 1.27)
+				)
+				(hide yes)
 			)
 		)
@@
 			)
 		)
+		(property "Silkscreen Value" "100k▶"
+			(at 53.34 50.8 90)
+			(effects
+				(font
+					(size 1.27 1.27)
+				)
+				(hide yes)
+			)
+		)
 		(pin "1"
 		)
@@
 		)
 		(property "Description" "Polarized capacitor"
+			(at 57.15 121.92 0)
+			(effects
+				(font
+					(size 1.27 1.27)
+				)
+				(hide yes)
+			)
+		)
+		(property "Silkscreen Value" "22uF▶"
 			(at 57.15 121.92 0)
 			(effects
@@
 			(at 57.15 134.62 0)
 			(effects
+				(font
+					(size 1.27 1.27)
+				)
+				(hide yes)
+			)
+		)
+		(property "Silkscreen Value" "◀22uF"
+			(at 57.15 134.62 0)
+			(effects

Commit message: added BuildNotes.md. Removed production folder
Parts:
- C13: Silkscreen Value 104▼ -> 104▶
- C5: Silkscreen Value 104▲ -> ◀104
- POT1: footprint PCM_4ms_Potentiometer:Potentiometer_Alps_RK09L_Double_Vertical -> Library:Dual_9mm_Potentiometer_50K_RK1114GH; Display 50k -> Dual 50k
- R5: footprint Resistor_THT:R_Axial_DIN0204_L3.6mm_D1.6mm_P5.08mm_Horizontal -> Resistor_THT:R_Axial_DIN0204_L3.6mm_D1.6mm_P1.90mm_Vertical; Silkscreen Value (none) -> 100k▶
- R7: footprint Resistor_THT:R_Axial_DIN0204_L3.6mm_D1.6mm_P5.08mm_Horizontal -> Resistor_THT:R_Axial_DIN0204_L3.6mm_D1.6mm_P1.90mm_Vertical; Silkscreen Value (none) -> 1k▼
- R8: footprint Resistor_THT:R_Axial_DIN0204_L3.6mm_D1.6mm_P5.08mm_Horizontal -> Resistor_THT:R_Axial_DIN0204_L3.6mm_D1.6mm_P1.90mm_Vertical; Silkscreen Value (none) -> ◀1k
Changed lines of the file:
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@@
 			)
 		)
-		(property "Footprint" "PCM_4ms_Potentiometer:Potentiometer_Alps_RK09L_Double_Vertical"
+		(property "Footprint" "Library:Dual_9mm_Potentiometer_50K_RK1114GH"
 			(at 138.43 66.04 0)
 			(effects
@@
 			)
 		)
-		(property "Description" "50k Linear, 9mm pot, Dual, D-Shaft, Dual Row"
+		(property "Description" "VOLUME"
 			(at 133.35 59.69 0)
 			(effects
@@
 			)
 		)
-		(property "Display" "50k"
+		(property "Display" "Dual 50k"
 			(at 137.16 59.6899 0)
 			(effects
@@
 			)
 		)
-		(property "Footprint" "PCM_4ms_Potentiometer:Potentiometer_Alps_RK09L_Double_Vertical"
+		(property "Footprint" "Library:Dual_9mm_Potentiometer_50K_RK1114GH"
 			(at 137.16 38.1 0)
 			(effects
@@
 			)
 		)
-		(property "Description" "50k Linear, 9mm pot, Dual, D-Shaft, Dual Row"
+		(property "Description" "VOLUME"
 			(at 132.08 31.75 0)
 			(effects
@@
 			)
 		)
-		(property "Display" "50k"
+		(property "Display" "Dual 50k"
 			(at 129.54 33.0199 0)
 			(effects
@@
 			)
 		)
-		(property "Footprint" "Resistor_THT:R_Axial_DIN0204_L3.6mm_D1.6mm_P5.08mm_Horizontal"
+		(property "Footprint" "Resistor_THT:R_Axial_DIN0204_L3.6mm_D1.6mm_P1.90mm_Vertical"
 			(at 114.3 76.708 90)
 			(effects
@@
 			)
 		)
+		(property "Silkscreen Value" "◀1k"
+			(at 114.3 74.93 90)
+			(effects
+				(font
+					(size 1.27 1.27)
+				)
+				(hide yes)
+			)
+		)
 		(pin "1"
 		)
@@
 			)
 		)
-		(property "Silkscreen Value" "104▲"
+		(property "Silkscreen Value" "◀104"
 			(at 72.39 121.92 0)
 			(effects
@@
 			)
 		)
-		(property "Footprint" "PCM_4ms_Potentiometer:Potentiometer_Alps_RK09L_Double_Vertical"
+		(property "Footprint" "Library:Dual_9mm_Potentiometer_50K_RK1114GH"
 			(at 137.16 85.09 0)
 			(effects
@@
 			)
 		)
-		(property "Description" "50k Linear, 9mm pot, Dual, D-Shaft, Dual Row"
+		(property "Description" "VOLUME"
 			(at 132.08 78.74 0)
 			(effects
@@
 			)
 		)
-		(property "Display" "50k"
+		(property "Display" "Dual 50k"
 			(at 129.54 80.0099 0)
 			(effects
@@
 			)
 		)
-		(property "Silkscreen Value" "104▼"
+		(property "Silkscreen Value" "104▶"
 			(at 139.7 31.75 0)
 			(effects
@@
 			)
 		)
-		(property "Footprint" "Resistor_THT:R_Axial_DIN0204_L3.6mm_D1.6mm_P5.08mm_Horizontal"
+		(property "Footprint" "Resistor_THT:R_Axial_DIN0204_L3.6mm_D1.6mm_P1.90mm_Vertical"
 			(at 114.3 29.718 90)
 			(effects
@@
 			)
 		)
+		(property "Silkscreen Value" "1k▼"
+			(at 114.3 27.94 90)
+			(effects
+				(font
+					(size 1.27 1.27)
+				)
+				(hide yes)
+			)
+		)
 		(pin "1"
 		)
@@
 			)
 		)
-		(property "Footprint" "Resistor_THT:R_Axial_DIN0204_L3.6mm_D1.6mm_P5.08mm_Horizontal"
+		(property "Footprint" "Resistor_THT:R_Axial_DIN0204_L3.6mm_D1.6mm_P1.90mm_Vertical"
 			(at 93.98 57.658 90)
 			(effects
@@
 			(effects
 				(font
+					(size 1.27 1.27)
+				)
+				(hide yes)
+			)
+		)
+		(property "Silkscreen Value" "100k▶"
+			(at 93.98 55.88 90)
+			(effects
+				(font

Commit message: v1.1 ready for final check
Parts:
- C1: footprint Capacitor_THT:CP_Radial_D4.0mm_P1.50mm -> Capacitor_THT:CP_Radial_D4.0mm_P2.00mm; Silkscreen Value 22uF▶ -> ◀22uF
- C10, C9: Silkscreen Value 104▶ -> 104▲
- C13: Silkscreen Value 104▶ -> ◀104
- C14: Silkscreen Value ▲104 -> 104▶
- C2: footprint Capacitor_THT:CP_Radial_D4.0mm_P1.50mm -> Capacitor_THT:CP_Radial_D4.0mm_P2.00mm; Silkscreen Value ◀22uF -> 22uF▶
- C6, C7: Silkscreen Value 104▼ -> 104▲
- IC1: Silkscreen Value (none) -> NJM4556AD▲
- IC2: Silkscreen Value (none) -> NJM4556AD▼
- POT1: Display Dual 50k -> Dual 50k B
- R1: footprint Resistor_THT:R_Axial_DIN0204_L3.6mm_D1.6mm_P5.08mm_Horizontal -> Resistor_THT:R_Axial_DIN0204_L3.6mm_D1.6mm_P1.90mm_Vertical; Silkscreen Value 100k▶ -> 100k▼
- R10: footprint Resistor_THT:R_Axial_DIN0204_L3.6mm_D1.6mm_P5.08mm_Horizontal -> Resistor_THT:R_Axial_DIN0204_L3.6mm_D1.6mm_P1.90mm_Vertical; Silkscreen Value (none) -> 100k▲
- R11, R12: value 1 -> 1Ω; footprint Resistor_THT:R_Axial_DIN0204_L3.6mm_D1.6mm_P5.08mm_Horizontal -> Resistor_THT:R_Axial_DIN0204_L3.6mm_D1.6mm_P1.90mm_Vertical; Silkscreen Value (none) -> 1Ω
- R13, R14: value 1 -> 1Ω; footprint Resistor_THT:R_Axial_DIN0204_L3.6mm_D1.6mm_P5.08mm_Horizontal -> Resistor_THT:R_Axial_DIN0204_L3.6mm_D1.6mm_P1.90mm_Vertical; Silkscreen Value (none) -> 1Ω▼
- R2: footprint Resistor_THT:R_Axial_DIN0204_L3.6mm_D1.6mm_P5.08mm_Horizontal -> Resistor_THT:R_Axial_DIN0204_L3.6mm_D1.6mm_P1.90mm_Vertical; Silkscreen Value 100k▶ -> ◀100k
- R3: footprint Resistor_THT:R_Axial_DIN0204_L3.6mm_D1.6mm_P5.08mm_Horizontal -> Resistor_THT:R_Axial_DIN0204_L3.6mm_D1.6mm_P1.90mm_Vertical; Silkscreen Value (none) -> ◀100k
- R4, R6: footprint Resistor_THT:R_Axial_DIN0204_L3.6mm_D1.6mm_P5.08mm_Horizontal -> Resistor_THT:R_Axial_DIN0204_L3.6mm_D1.6mm_P1.90mm_Vertical; Silkscreen Value (none) -> 100k▶
- R5: Silkscreen Value 100k▶ -> ◀100k
- R7: Silkscreen Value 1k▼ -> ◀1k
- R8: Silkscreen Value ◀1k -> 1k▶
- R9: footprint Resistor_THT:R_Axial_DIN0204_L3.6mm_D1.6mm_P5.08mm_Horizontal -> Resistor_THT:R_Axial_DIN0204_L3.6mm_D1.6mm_P1.90mm_Vertical; Silkscreen Value (none) -> 100k▼
- U1, U2: Silkscreen Value (none) -> LME49720▲
Changed lines of the file:
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@@
 			)
 		)
-		(property "Footprint" "Resistor_THT:R_Axial_DIN0204_L3.6mm_D1.6mm_P5.08mm_Horizontal"
+		(property "Footprint" "Resistor_THT:R_Axial_DIN0204_L3.6mm_D1.6mm_P1.90mm_Vertical"
 			(at 93.98 104.648 90)
 			(effects
@@
 			)
 		)
+		(property "Silkscreen Value" "100k▶"
+			(at 93.98 102.87 0)
+			(effects
+				(font
+					(size 1.27 1.27)
+				)
+				(hide yes)
+			)
+		)
 		(pin "1"
 		)
@@
 			)
 		)
-		(property "Silkscreen Value" "104▼"
+		(property "Silkscreen Value" "104▲"
 			(at 72.39 134.62 0)
 			(effects
@@
 			)
 		)
-		(property "Footprint" "Resistor_THT:R_Axial_DIN0204_L3.6mm_D1.6mm_P5.08mm_Horizontal"
+		(property "Footprint" "Resistor_THT:R_Axial_DIN0204_L3.6mm_D1.6mm_P1.90mm_Vertical"
 			(at 147.828 83.82 90)
 			(effects
@@
 			)
 		)
+		(property "Silkscreen Value" "100k▲"
+			(at 146.05 83.82 0)
+			(effects
+				(font
+					(size 1.27 1.27)
+				)
+				(hide yes)
+			)
+		)
 		(pin "1"
 		)
@@
 			)
 		)
-		(property "Display" "Dual 50k"
+		(property "Display" "Dual 50k B"
 			(at 137.16 59.6899 0)
 			(effects
@@
 			)
 		)
+		(property "Silkscreen Value" "LME49720▲"
+			(at 92.71 74.93 0)
+			(effects
+				(font
+					(size 1.27 1.27)
+				)
+				(hide yes)
+			)
+		)
 		(pin "4"
 		)
@@
 			)
 		)
-		(property "Silkscreen Value" "104▶"
+		(property "Silkscreen Value" "104▲"
 			(at 87.63 121.92 0)
 			(effects
@@
 			)
 		)
-		(property "Display" "Dual 50k"
+		(property "Display" "Dual 50k B"
 			(at 129.54 33.0199 0)
 			(effects
@@
 			)
 		)
-		(property "Silkscreen Value" "◀1k"
+		(property "Silkscreen Value" "1k▶"
 			(at 114.3 74.93 90)
 			(effects
@@
 			)
 		)
+		(property "Silkscreen Value" "LME49720▲"
+			(at 54.61 30.48 0)
+			(effects
+				(font
+					(size 1.27 1.27)
+				)
+				(hide yes)
+			)
+		)
 		(pin "4"
 		)
@@
 			)
 		)
-		(property "Footprint" "Resistor_THT:R_Axial_DIN0204_L3.6mm_D1.6mm_P5.08mm_Horizontal"
+		(property "Footprint" "Resistor_THT:R_Axial_DIN0204_L3.6mm_D1.6mm_P1.90mm_Vertical"
 			(at 76.2 79.248 90)
 			(effects
@@
 			)
 		)
+		(property "Silkscreen Value" "100k▶"
+			(at 76.2 77.47 0)
+			(effects
+				(font
+					(size 1.27 1.27)
+				)
+				(hide yes)
+			)
+		)
 		(pin "1"
 		)
@@
 			)
 		)
-		(property "Footprint" "Resistor_THT:R_Axial_DIN0204_L3.6mm_D1.6mm_P5.08mm_Horizontal"
+		(property "Footprint" "Resistor_THT:R_Axial_DIN0204_L3.6mm_D1.6mm_P1.90mm_Vertical"
 			(at 76.2 32.258 90)
 			(effects
@@
 			)
 		)
+		(property "Silkscreen Value" "◀100k"
+			(at 76.2 30.48 0)
+			(effects
+				(font
+					(size 1.27 1.27)
+				)
+				(hide yes)
+			)
+		)
 		(pin "1"
 		)
@@
 			)
 		)
-		(property "Silkscreen Value" "▲104"
+		(property "Silkscreen Value" "104▶"
 			(at 139.7 78.74 0)
 			(effects
@@
 			)
 		)
-		(property "Display" "Dual 50k"
+		(property "Display" "Dual 50k B"
 			(at 129.54 80.0099 0)
 			(effects
@@
 			)
 		)
-		(property "Silkscreen Value" "104▶"
+		(property "Silkscreen Value" "104▲"
 			(at 87.63 134.62 0)
 			(effects
@@
 			)
 		)
+		(property "Silkscreen Value" "NJM4556AD▼"
+			(at 152.4 73.66 0)
+			(effects
+				(font
+					(size 1.27 1.27)
+				)
+				(hide yes)
+			)
+		)
 		(pin "5"
 		)
@@
 			)
 		)
-		(property "Value" "1"
+		(property "Value" "1Ω"
 			(at 199.39 29.21 90)
 			(effects
@@
 			)
 		)
-		(property "Footprint" "Resistor_THT:R_Axial_DIN0204_L3.6mm_D1.6mm_P5.08mm_Horizontal"
+		(property "Footprint" "Resistor_THT:R_Axial_DIN0204_L3.6mm_D1.6mm_P1.90mm_Vertical"
 			(at 199.39 30.988 90)
 			(effects
@@
 			)
 		)
+		(property "Silkscreen Value" "1Ω"
+			(at 199.39 29.21 0)
+			(effects
+				(font
+					(size 1.27 1.27)
+				)
+				(hide yes)
+			)
+		)
 		(pin "1"
 		)
@@
 			)
 		)
-		(property "Silkscreen Value" "104▶"
+		(property "Silkscreen Value" "◀104"
 			(at 139.7 31.75 0)
 			(effects
@@
 			)
 		)
+		(property "Silkscreen Value" "NJM4556AD▲"
+			(at 152.4 26.67 0)
+			(effects
+				(font
+					(size 1.27 1.27)
+				)
+				(hide yes)
+			)
+		)
 		(pin "5"
 		)
@@
 			)
 		)
-		(property "Value" "1"
+		(property "Value" "1Ω"
 			(at 199.39 67.31 90)
 			(effects
@@
 			)
 		)
-		(property "Footprint" "Resistor_THT:R_Axial_DIN0204_L3.6mm_D1.6mm_P5.08mm_Horizontal"
+		(property "Footprint" "Resistor_THT:R_Axial_DIN0204_L3.6mm_D1.6mm_P1.90mm_Vertical"
 			(at 199.39 69.088 90)
 			(effects
@@
 			)
 		)
+		(property "Silkscreen Value" "1Ω▼"
+			(at 199.39 67.31 0)
+			(effects
+				(font
+					(size 1.27 1.27)
+				)
+				(hide yes)
+			)
+		)
 		(pin "1"
 		)
@@
 			)
 		)
-		(property "Silkscreen Value" "104▼"
+		(property "Silkscreen Value" "104▲"
 			(at 80.01 121.92 0)
 			(effects
@@
 			)
 		)
-		(property "Footprint" "Resistor_THT:R_Axial_DIN0204_L3.6mm_D1.6mm_P5.08mm_Horizontal"
+		(property "Footprint" "Resistor_THT:R_Axial_DIN0204_L3.6mm_D1.6mm_P1.90mm_Vertical"
 			(at 53.34 55.372 90)
 			(effects
@@
 			)
 		)
-		(property "Silkscreen Value" "100k▶"
+		(property "Silkscreen Value" "◀100k"
 			(at 53.34 57.15 90)
 			(effects
@@
 			)
 		)
-		(property "Footprint" "Resistor_THT:R_Axial_DIN0204_L3.6mm_D1.6mm_P5.08mm_Horizontal"
+		(property "Footprint" "Resistor_THT:R_Axial_DIN0204_L3.6mm_D1.6mm_P1.90mm_Vertical"
 			(at 53.34 52.578 90)
 			(effects
@@
 			)
 		)
-		(property "Silkscreen Value" "100k▶"
+		(property "Silkscreen Value" "100k▼"
 			(at 53.34 50.8 90)
 			(effects
@@
 			)
 		)
-		(property "Footprint" "Capacitor_THT:CP_Radial_D4.0mm_P1.50mm"
+		(property "Footprint" "Capacitor_THT:CP_Radial_D4.0mm_P2.00mm"
 			(at 58.1152 125.73 0)
 			(effects
@@
 			)
 		)
-		(property "Silkscreen Value" "22uF▶"
+		(property "Silkscreen Value" "◀22uF"
 			(at 57.15 121.92 0)
 			(effects
@@
 			)
 		)
-		(property "Silkscreen Value" "1k▼"
+		(property "Silkscreen Value" "◀1k"
 			(at 114.3 27.94 90)
 			(effects
@@
 			)
 		)
-		(property "Value" "1"
+		(property "Value" "1Ω"
 			(at 199.39 20.32 90)
 			(effects
@@
 			)
 		)
-		(property "Footprint" "Resistor_THT:R_Axial_DIN0204_L3.6mm_D1.6mm_P5.08mm_Horizontal"
+		(property "Footprint" "Resistor_THT:R_Axial_DIN0204_L3.6mm_D1.6mm_P1.90mm_Vertical"
 			(at 199.39 22.098 90)
 			(effects
@@
 			)
 		)
+		(property "Silkscreen Value" "1Ω"
+			(at 199.39 20.32 0)
+			(effects
+				(font
+					(size 1.27 1.27)
+				)
+				(hide yes)
+			)
+		)
 		(pin "1"
 		)
@@
 			)
 		)
-		(property "Footprint" "Resistor_THT:R_Axial_DIN0204_L3.6mm_D1.6mm_P5.08mm_Horizontal"
+		(property "Footprint" "Resistor_THT:R_Axial_DIN0204_L3.6mm_D1.6mm_P1.90mm_Vertical"
 			(at 147.828 36.83 90)
 			(effects
@@
 			)
 		)
+		(property "Silkscreen Value" "100k▼"
+			(at 146.05 36.83 0)
+			(effects
+				(font
+					(size 1.27 1.27)
+				)
+				(hide yes)
+			)
+		)
 		(pin "1"
 		)
@@
 			)
 		)
-		(property "Footprint" "Capacitor_THT:CP_Radial_D4.0mm_P1.50mm"
+		(property "Footprint" "Capacitor_THT:CP_Radial_D4.0mm_P2.00mm"
 			(at 58.1152 138.43 0)
 			(effects
@@
 			)
 		)
-		(property "Silkscreen Value" "◀22uF"
+		(property "Silkscreen Value" "22uF▶"
 			(at 57.15 134.62 0)
 			(effects
@@
 			)
 		)
-		(property "Value" "1"
+		(property "Value" "1Ω"
 			(at 199.39 76.2 90)
 			(effects
@@
 			)
 		)
-		(property "Footprint" "Resistor_THT:R_Axial_DIN0204_L3.6mm_D1.6mm_P5.08mm_Horizontal"
+		(property "Footprint" "Resistor_THT:R_Axial_DIN0204_L3.6mm_D1.6mm_P1.90mm_Vertical"
 			(at 199.39 77.978 90)
 			(effects
@@
 			)
 		)
+		(property "Silkscreen Value" "1Ω▼"
+			(at 199.39 76.2 0)
+			(effects
+				(font
+					(size 1.27 1.27)
+				)
+				(hide yes)
+			)
+		)
 		(pin "1"
 		)
@@
 			)
 		)
+		(property "Silkscreen Value" "LME49720▲"
+			(at 92.71 27.94 0)
+			(effects
+				(font
+					(size 1.27 1.27)
+				)
+				(hide yes)
+			)
+		)
 		(pin "4"
 		)
@@
 			)
 		)
-		(property "Silkscreen Value" "100k▶"
+		(property "Silkscreen Value" "◀100k"
 			(at 93.98 55.88 90)
 			(effects
@@
 			(at 54.61 77.47 0)
 			(effects
+				(font
+					(size 1.27 1.27)
+				)
+				(hide yes)
+			)
+		)
+		(property "Silkscreen Value" "LME49720▲"
+			(at 54.61 77.47 0)
+			(effects

Commit message: fixed silkscreening issues before sending for new boards
Parts:
- C10, C3: Silkscreen Value 104▲ -> 104▶
- C5: Silkscreen Value ◀104 -> ▼104
- C8: Silkscreen Value 104▼ -> 104▶
- R11, R12: Silkscreen Value 1Ω -> 1Ω▶
- R13: Silkscreen Value 1Ω▼ -> ▼1Ω
- R4: Silkscreen Value 100k▶ -> 100k▲
Changed lines of the file:
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@@
 			)
 		)
-		(property "Silkscreen Value" "100k▶"
+		(property "Silkscreen Value" "100k▲"
 			(at 76.2 77.47 0)
 			(effects
@@
 			)
 		)
-		(property "Silkscreen Value" "◀104"
+		(property "Silkscreen Value" "▼104"
 			(at 72.39 121.92 0)
 			(effects
@@
 			)
 		)
-		(property "Silkscreen Value" "104▲"
+		(property "Silkscreen Value" "104▶"
 			(at 87.63 134.62 0)
 			(effects
@@
 			)
 		)
-		(property "Silkscreen Value" "1Ω"
+		(property "Silkscreen Value" "1Ω▶"
 			(at 199.39 29.21 0)
 			(effects
@@
 			)
 		)
-		(property "Silkscreen Value" "1Ω▼"
+		(property "Silkscreen Value" "▼1Ω"
 			(at 199.39 67.31 0)
 			(effects
@@
 			)
 		)
-		(property "Silkscreen Value" "104▲"
+		(property "Silkscreen Value" "104▶"
 			(at 64.77 121.92 0)
 			(effects
@@
 			)
 		)
-		(property "Silkscreen Value" "104▼"
+		(property "Silkscreen Value" "104▶"
 			(at 80.01 134.62 0)
 			(effects
@@
 			)
 		)
-		(property "Silkscreen Value" "1Ω"
+		(property "Silkscreen Value" "1Ω▶"
 			(at 199.39 20.32 0)
 			(effects
